Commit message: Update cavepi.urdf.xacro

File: auv_dt/cavepi_description/urdf/cavepi.urdf.xacro (robot description, xacro)
@@ -41,5 +41,5 @@
         <inertial>
             <origin xyz="${scale_size*-0.8e-3} 0 ${scale_size*-4.55e-3}" rpy="0 0 0" />
-            <mass value="8.5" />
+            <mass value="8.714" />
             <inertia ixx="41763721.74e-9" ixy="76.64e-9" ixz="-1071029.52e-9"
                      iyy="99391057.27e-9" iyz="603.74e-9"

Commit message: Update cavepi.urdf.xacro

File: auv_dt/cavepi_description/urdf/cavepi.urdf.xacro (robot description, xacro)
@@ -26,5 +26,5 @@
         <visual>
             <geometry>
-                <mesh filename="package://nemogator_description/meshes/main_body_link_cavepi.STL"
+                <mesh filename="package://cavepi_description/meshes/main_body_link_cavepi.STL"
                       scale="${scale_size} ${scale_size} ${scale_size}" />
             </geometry>
@@ -34,5 +34,5 @@
         <collision>
             <geometry>
-                <mesh filename="package://nemogator_description/meshes/main_body_link_cavepi.STL"
+                <mesh filename="package://cavepi_description/meshes/main_body_link_cavepi.STL"
                       scale="${scale_size} ${scale_size} ${scale_size}" />
             </geometry>
@@ -57,5 +57,5 @@
         <visual>
             <geometry>
-                <mesh filename="package://nemogator_description/meshes/front_right_thruster_link_cavepi.STL"
+                <mesh filename="package://cavepi_description/meshes/front_right_thruster_link_cavepi.STL"
                       scale="${scale_size} ${scale_size} ${scale_size}" />
             </geometry>
@@ -65,5 +65,5 @@
         <collision>
             <geometry>
-                <mesh filename="package://nemogator_description/meshes/front_right_thruster_link_cavepi.STL"
+                <mesh filename="package://cavepi_description/meshes/front_right_thruster_link_cavepi.STL"
                       scale="${scale_size} ${scale_size} ${scale_size}" />
             </geometry>
@@ -89,5 +89,5 @@
         <visual>
             <geometry>
-                <mesh filename="package://nemogator_description/meshes/front_left_thruster_link_cavepi.STL"
+                <mesh filename="package://cavepi_description/meshes/front_left_thruster_link_cavepi.STL"
                       scale="${scale_size} ${scale_size} ${scale_size}" />
             </geometry>
@@ -97,5 +97,5 @@
         <collision>
             <geometry>
-                <mesh filename="package://nemogator_description/meshes/front_left_thruster_link_cavepi.STL"
+                <mesh filename="package://cavepi_description/meshes/front_left_thruster_link_cavepi.STL"
                       scale="${scale_size} ${scale_size} ${scale_size}" />
             </geometry>
@@ -121,5 +121,5 @@
         <visual>
             <geometry>
-                <mesh filename="package://nemogator_description/meshes/rear_right_thruster_link_cavepi.STL"
+                <mesh filename="package://cavepi_description/meshes/rear_right_thruster_link_cavepi.STL"
                       scale="${scale_size} ${scale_size} ${scale_size}" />
             </geometry>
@@ -129,5 +129,5 @@
         <collision>
             <geometry>
-                <mesh filename="package://nemogator_description/meshes/rear_right_thruster_link_cavepi.STL"
+                <mesh filename="package://cavepi_description/meshes/rear_right_thruster_link_cavepi.STL"
                       scale="${scale_size} ${scale_size} ${scale_size}" />
             </geometry>
@@ -153,5 +153,5 @@
         <visual>
             <geometry>
-                <mesh filename="package://nemogator_description/meshes/rear_left_thruster_link_cavepi.STL"
+                <mesh filename="package://cavepi_description/meshes/rear_left_thruster_link_cavepi.STL"
                       scale="${scale_size} ${scale_size} ${scale_size}" />
             </geometry>
@@ -161,5 +161,5 @@
         <collision>
             <geometry>
-                <mesh filename="package://nemogator_description/meshes/rear_left_thruster_link_cavepi.STL"
+                <mesh filename="package://cavepi_description/meshes/rear_left_thruster_link_cavepi.STL"
                       scale="${scale_size} ${scale_size} ${scale_size}" />
             </geometry>

Commit message: Update cavepi.urdf.xacro

File: auv_dt/cavepi_description/urdf/cavepi.urdf.xacro (robot description, xacro)
@@ -45,5 +45,5 @@
         <inertial>
             <origin xyz="${scale_size*-0.8e-3} 0 ${scale_size*-4.55e-3}" rpy="0 0 0" />
-            <mass value="8.714" />
+            <mass value="8.6" />
             <inertia ixx="41763721.74e-9" ixy="76.64e-9" ixz="-1071029.52e-9"
                      iyy="99391057.27e-9" iyz="603.74e-9"
